File: hardware/clockgen/low+high_voltage/STM_Morpho.sch (KiCad schematic (older format))
At the start: 32 parts, among them CN10 Conn_02x19_Odd_Even, CN7 Conn_02x19_Odd_Even, J1 Conn_02x20_Odd_Even, J2 Conn_02x20_Odd_Even, U1 74ALVC164245DLG4, U10 CD40109BNSR, U2 74ALVC164245DLG4, U3 CD40109BNSR, U4 CD40109BNSR, U5 CD40109BNSR, U6 CD40109BNSR, U7 CD40109BNSR, U8 CD40109BNSR, U9 CD40109BNSR

Commit message: Two PCBs are routed
Parts:
- removed J1, J2: Conn_02x20_Odd_Even, Connector_PinHeader_2.54mm:PinHeader_2x20_P2.54mm_Vertical, symbol Connector_Generic:Conn_02x20_Counter_Clockwise
- added J1, J2: Conn_02x20_Counter_Clockwise, Connector_PinHeader_2.54mm:PinHeader_2x20_P2.54mm_Vertical, symbol Connector_Generic:Conn_02x20_Odd_Even
- U1, U2: symbol 2021-08-26_08-32-07:74ALVC164245DLG4 -> STM_Morpho-rescue:74ALVC164245DLG4-2021-08-26_08-32-07
- U10, U3, U4, U5, U6, U7, U8, U9: symbol 2021-08-27_11-58-03:CD40109BNSR -> STM_Morpho-rescue:CD40109BNSR-2021-08-27_11-58-03
Connections:
- net +15V: now also J1.37 (Pin_37), J1.39 (Pin_39)
- net +3V3: now also J1.3 (Pin_3), J2.3 (Pin_3)
- net +5V: now also J1.1 (Pin_1), J2.1 (Pin_1)
- net GND: now also J1.2 (Pin_2), J1.38 (Pin_38), J1.4 (Pin_4), J1.40 (Pin_40), J2.2 (Pin_2), J2.38 (Pin_38), J2.4 (Pin_4), J2.40 (Pin_40)
- net NC: now also J2.37 (Pin_37), J2.39 (Pin_39)
- net PA0_5V: now also J2.13 (Pin_13)
- net PA0_HIGH: now also J1.13 (Pin_13)
- net PA10_5V: now also J2.5 (Pin_5)
- net PA10_HIGH: now also J1.5 (Pin_5)
- net PA11_5V: now also J2.8 (Pin_8)
- net PA11_HIGH: now also J1.34 (Pin_34)
- net PA12_5V: now also J2.10 (Pin_10)
- net PA12_HIGH: now also J1.32 (Pin_32)
- net PA13_5V: now also J2.12 (Pin_12)
- net PA13_HIGH: now also J1.30 (Pin_30)
- net PA14_5V: now also J2.14 (Pin_14)
- net PA14_HIGH: now also J1.28 (Pin_28)
- net PA15_5V: now also J2.16 (Pin_16)
- net PA15_HIGH: now also J1.26 (Pin_26)
- net PA1_5V: now also J2.25 (Pin_25)
- net PA1_HIGH: now also J1.25 (Pin_25)
- net PA2_5V: now also J2.27 (Pin_27)
- net PA2_HIGH: now also J1.27 (Pin_27)
- net PA3_5V: now also J2.29 (Pin_29)
- net PA3_HIGH: now also J1.29 (Pin_29)
- net PA4_5V: now also J2.31 (Pin_31)
- net PA4_HIGH: now also J1.31 (Pin_31)
- net PA5_5V: now also J2.33 (Pin_33)
- net PA5_HIGH: now also J1.33 (Pin_33)
- net PA6_5V: now also J2.21 (Pin_21)
- net PA6_HIGH: now also J1.21 (Pin_21)
- net PA7_5V: now also J2.23 (Pin_23)
- net PA7_HIGH: now also J1.23 (Pin_23)
- net PA8_5V: now also J2.35 (Pin_35)
- net PA8_HIGH: now also J1.35 (Pin_35)
- net PA9_5V: now also J2.6 (Pin_6)
- net PA9_HIGH: now also J1.36 (Pin_36)
- net PB10_5V: now also J2.7 (Pin_7)
- net PB10_HIGH: now also J1.7 (Pin_7)
- net PB5_5V: now also J2.9 (Pin_9)
- net PB5_HIGH: now also J1.9 (Pin_9)
- net PB6_5V: now also J2.11 (Pin_11)
- net PB6_HIGH: now also J1.11 (Pin_11)
- net PB8_5V: now also J2.17 (Pin_17)
- net PB8_HIGH: now also J1.17 (Pin_17)
- net PB9_5V: now also J2.19 (Pin_19)
- net PB9_HIGH: now also J1.19 (Pin_19)
- net PC0_5V: now also J2.18 (Pin_18)
- net PC0_HIGH: now also J1.24 (Pin_24)
- net PC10_5V: now also J2.36 (Pin_36)
- net PC10_HIGH: now also J1.6 (Pin_6)
- net PC1_5V: now also J2.20 (Pin_20)
- net PC1_HIGH: now also J1.22 (Pin_22)
- net PC2_5V: now also J2.22 (Pin_22)
- net PC2_HIGH: now also J1.20 (Pin_20)
- net PC3_5V: now also J2.24 (Pin_24)
- net PC3_HIGH: now also J1.18 (Pin_18)
- net PC4_5V: now also J2.26 (Pin_26)
- net PC4_HIGH: now also J1.16 (Pin_16)
- net PC5_5V: now also J2.28 (Pin_28)
- net PC5_HIGH: now also J1.14 (Pin_14)
- net PC6_5V: now also J2.30 (Pin_30)
- net PC6_HIGH: now also J1.12 (Pin_12)
- net PC7_5V: now also J2.15 (Pin_15)
- net PC7_HIGH: now also J1.15 (Pin_15)
- net PC8_5V: now also J2.32 (Pin_32)
- net PC8_HIGH: now also J1.10 (Pin_10)
- net PC9_5V: now also J2.34 (Pin_34)
- net PC9_HIGH: now also J1.8 (Pin_8)
Changed lines of the file:
@@
 PA3
 $Comp
-L 2021-08-26_08-32-07:74ALVC164245DLG4 U1
+L STM_Morpho-rescue:74ALVC164245DLG4-2021-08-26_08-32-07 U1
 U 1 1 6128B1C2
 P 4400 1050
@@
 PULLUP
 $Comp
-L 2021-08-26_08-32-07:74ALVC164245DLG4 U2
+L STM_Morpho-rescue:74ALVC164245DLG4-2021-08-26_08-32-07 U2
 U 1 1 6130056B
 P 8750 1050
@@
 $EndComp
 $Comp
-L 2021-08-27_11-58-03:CD40109BNSR U3
+L STM_Morpho-rescue:CD40109BNSR-2021-08-27_11-58-03 U3
 U 1 1 613E344D
 P 1550 4950
@@
 PULLUP_HIGH
 $Comp
-L 2021-08-27_11-58-03:CD40109BNSR U4
+L STM_Morpho-rescue:CD40109BNSR-2021-08-27_11-58-03 U4
 U 1 1 613FF819
 P 1550 6650
@@
 PULLUP_HIGH
 $Comp
-L 2021-08-27_11-58-03:CD40109BNSR U5
+L STM_Morpho-rescue:CD40109BNSR-2021-08-27_11-58-03 U5
 U 1 1 61400961
 P 1550 8200
@@
 PULLUP_HIGH
 $Comp
-L 2021-08-27_11-58-03:CD40109BNSR U6
+L STM_Morpho-rescue:CD40109BNSR-2021-08-27_11-58-03 U6
 U 1 1 614016CB
 P 1600 9800
@@
 PULLUP_HIGH
 $Comp
-L 2021-08-27_11-58-03:CD40109BNSR U7
+L STM_Morpho-rescue:CD40109BNSR-2021-08-27_11-58-03 U7
 U 1 1 6141034C
 P 5900 4950
@@
 PULLUP_HIGH
 $Comp
-L 2021-08-27_11-58-03:CD40109BNSR U8
+L STM_Morpho-rescue:CD40109BNSR-2021-08-27_11-58-03 U8
 U 1 1 61410359
 P 5900 6650
@@
 PULLUP_HIGH
 $Comp
-L 2021-08-27_11-58-03:CD40109BNSR U9
+L STM_Morpho-rescue:CD40109BNSR-2021-08-27_11-58-03 U9
 U 1 1 61410366
 P 5900 8200
@@
 PULLUP_HIGH
 $Comp
-L 2021-08-27_11-58-03:CD40109BNSR U10
+L STM_Morpho-rescue:CD40109BNSR-2021-08-27_11-58-03 U10
 U 1 1 61410373
 P 5950 9800
@@
 Text Label 8750 3250 2    50   ~ 0
 PC10_5V
-$Comp
-L Connector_Generic:Conn_02x20_Counter_Clockwise J1
-U 1 1 612BBAFC
-P 13000 1800
-F 0 "J1" H 13050 2917 50  0000 C CNN
-F 1 "Conn_02x20_Odd_Even" H 13050 2826 50  0000 C CNN
-F 2 "Connector_PinHeader_2.54mm:PinHeader_2x20_P2.54mm_Vertical" H 13000 1800 50  0001 C CNN
-F 3 "~" H 13000 1800 50  0001 C CNN
-	1    13000 1800
-	1    0    0    -1
-$EndComp
 Text Label 12800 2100 2    50   ~ 0
 PA1_5V
@@
 Text Label 12800 2600 2    50   ~ 0
 PA8_5V
-Text Label 13300 2600 0    50   ~ 0
+Text Label 13300 1100 2    50   ~ 0
 PA9_5V
-Text Label 13300 2500 0    50   ~ 0
+Text Label 13300 1200 2    50   ~ 0
 PA11_5V
-Text Label 13300 2400 0    50   ~ 0
-PA12_5V
-Text Label 13300 2300 0    50   ~ 0
+Text Label 13300 1400 2    50   ~ 0
 PA13_5V
-Text Label 13300 2200 0    50   ~ 0
+Text Label 13300 1500 2    50   ~ 0
 PA14_5V
-Text Label 13300 2100 0    50   ~ 0
+Text Label 13300 1600 2    50   ~ 0
 PA15_5V
-Text Label 13300 2000 0    50   ~ 0
+Text Label 13300 1700 2    50   ~ 0
 PC0_5V
-Text Label 13300 1900 0    50   ~ 0
+Text Label 13300 1800 2    50   ~ 0
 PC1_5V
-Text Label 13300 1800 0    50   ~ 0
+Text Label 13300 1900 2    50   ~ 0
 PC2_5V
-Text Label 13300 1700 0    50   ~ 0
+Text Label 13300 2000 2    50   ~ 0
 PC3_5V
-Text Label 13300 1600 0    50   ~ 0
+Text Label 13300 2100 2    50   ~ 0
 PC4_5V
-Text Label 13300 1500 0    50   ~ 0
+Text Label 13300 2200 2    50   ~ 0
 PC5_5V
-Text Label 13300 1400 0    50   ~ 0
+Text Label 13300 2300 2    50   ~ 0
 PC6_5V
-Text Label 13300 1300 0    50   ~ 0
+Text Label 13300 2400 2    50   ~ 0
 PC8_5V
-Text Label 13300 1200 0    50   ~ 0
+Text Label 13300 2500 2    50   ~ 0
 PC9_5V
-Text Label 13300 1100 0    50   ~ 0
+Text Label 13300 2600 2    50   ~ 0
 PC10_5V
 Text Label 12800 1000 2    50   ~ 0
@@
 Text Label 11750 5500 2    50   ~ 0
 PA7_HIGH
-$Comp
-L Connector_Generic:Conn_02x20_Counter_Clockwise J2
-U 1 1 61341D64
-P 11950 5300
-F 0 "J2" H 12000 6417 50  0000 C CNN
-F 1 "Conn_02x20_Odd_Even" H 12000 6326 50  0000 C CNN
-F 2 "Connector_PinHeader_2.54mm:PinHeader_2x20_P2.54mm_Vertical" H 11950 5300 50  0001 C CNN
-F 3 "~" H 11950 5300 50  0001 C CNN
-	1    11950 5300
-	1    0    0    -1
-$EndComp
 Text Label 11750 5600 2    50   ~ 0
 PA1_HIGH
@@
 Text Label 15300 7750 1    50   ~ 0
 GND
+$Comp
+L Connector_Generic:Conn_02x20_Odd_Even J2
+U 1 1 612AD630
+P 13000 1800
+F 0 "J2" H 13050 2917 50  0000 C CNN
+F 1 "Conn_02x20_Counter_Clockwise" H 13050 2826 50  0000 C CNN
+F 2 "Connector_PinHeader_2.54mm:PinHeader_2x20_P2.54mm_Vertical" H 13000 1800 50  0001 C CNN
+F 3 "~" H 13000 1800 50  0001 C CNN
+	1    13000 1800
+	1    0    0    -1
+$EndComp
+$Comp
+L Connector_Generic:Conn_02x20_Odd_Even J1
+U 1 1 612B30C2
+P 11950 5300
+F 0 "J1" H 12000 6417 50  0000 C CNN
+F 1 "Conn_02x20_Counter_Clockwise" H 12000 6326 50  0000 C CNN
+F 2 "Connector_PinHeader_2.54mm:PinHeader_2x20_P2.54mm_Vertical" H 11950 5300 50  0001 C CNN
+F 3 "~" H 11950 5300 50  0001 C CNN
+	1    11950 5300
+	1    0    0    -1
+$EndComp
+Text Label 13300 1300 2    50   ~ 0
+PA12_5V
 $EndSCHEMATC
