File: hardware/clockgen/high/STM_Morpho.sch (KiCad schematic (older format))
At the start: 32 parts, among them CN10 Conn_02x19_Odd_Even, CN7 Conn_02x19_Odd_Even, J1 Conn_02x20_Odd_Even, J2 Conn_02x20_Odd_Even, U1 74ALVC164245DLG4, U10 CD40109BNSR, U2 74ALVC164245DLG4, U3 CD40109BNSR, U4 CD40109BNSR, U5 CD40109BNSR, U6 CD40109BNSR, U7 CD40109BNSR, U8 CD40109BNSR, U9 CD40109BNSR

Commit message: Two PCBs are routed
Parts:
- removed C2: CP, Capacitor_THT:CP_Radial_D5.0mm_P2.00mm, symbol Device:CP
- removed C3.31, C3.32, C5V1, C5V2: C, Capacitor_SMD:C_0805_2012Metric, symbol Device:C
- removed CN10, CN7: Conn_02x19_Odd_Even, Connector_PinSocket_2.54mm:PinSocket_2x19_P2.54mm_Vertical, symbol Connector_Generic:Conn_02x19_Odd_Even
- removed J1, J2: Conn_02x20_Odd_Even, Connector_PinHeader_2.54mm:PinHeader_2x20_P2.54mm_Vertical, symbol Connector_Generic:Conn_02x20_Counter_Clockwise
- removed R1, R2: 10K, Resistor_THT:R_Axial_DIN0207_L6.3mm_D2.5mm_P2.54mm_Vertical, symbol Device:R
- removed U1, U2: 74ALVC164245DLG4, footprints:74ALVC164245DLG4, symbol 2021-08-26_08-32-07:74ALVC164245DLG4
- added J1, J2: Conn_02x20_Odd_Even, Connector_PinHeader_2.54mm:PinHeader_2x20_P2.54mm_Vertical, symbol Connector_Generic:Conn_02x20_Odd_Even
- added J3: Conn_01x02_Female, Connector_PinHeader_2.54mm:PinHeader_1x02_P2.54mm_Vertical, symbol Connector:Conn_01x02_Female
- U1: renamed from U3; symbol 2021-08-27_11-58-03:CD40109BNSR -> STM_Morpho-rescue:CD40109BNSR-2021-08-27_11-58-03
- U2: renamed from U4; symbol 2021-08-27_11-58-03:CD40109BNSR -> STM_Morpho-rescue:CD40109BNSR-2021-08-27_11-58-03
- U3: renamed from U5; symbol 2021-08-27_11-58-03:CD40109BNSR -> STM_Morpho-rescue:CD40109BNSR-2021-08-27_11-58-03
- U4: renamed from U6; symbol 2021-08-27_11-58-03:CD40109BNSR -> STM_Morpho-rescue:CD40109BNSR-2021-08-27_11-58-03
- U5: renamed from U7; symbol 2021-08-27_11-58-03:CD40109BNSR -> STM_Morpho-rescue:CD40109BNSR-2021-08-27_11-58-03
- U6: renamed from U8; symbol 2021-08-27_11-58-03:CD40109BNSR -> STM_Morpho-rescue:CD40109BNSR-2021-08-27_11-58-03
- U7: renamed from U9; symbol 2021-08-27_11-58-03:CD40109BNSR -> STM_Morpho-rescue:CD40109BNSR-2021-08-27_11-58-03
- U8: renamed from U10; symbol 2021-08-27_11-58-03:CD40109BNSR -> STM_Morpho-rescue:CD40109BNSR-2021-08-27_11-58-03
- renumbered C3 to C4, R3 to R1
Connections:
- net PA0 is gone; now on net PA0_5V: U2.3 (A)
- net PA1 is gone; now on net PA1_5V: U3.10 (C)
- net PA10 is gone; now on net PA10_5V: U1.3 (A)
- net PA11 is gone; now on net PA11_5V: U5.6 (B)
- net PA12 is gone; now on net PA12_5V: U5.10 (C)
- net PA13 is gone; now on net PA13_5V: U5.14 (D)
- net PA14 is gone; now on net PA14_5V: U6.3 (A)
- net PA15 is gone; now on net PA15_5V: U6.6 (B)
- net PA2 is gone; now on net PA2_5V: U3.14 (D)
- net PA3 is gone; now on net PA3_5V: U4.3 (A)
- net PA4 is gone; now on net PA4_5V: U4.6 (B)
- net PA5 is gone; now on net PA5_5V: U4.10 (C)
- net PA6 is gone; now on net PA6_5V: U3.3 (A)
- net PA7 is gone; now on net PA7_5V: U3.6 (B)
- net PA8 is gone; now on net PA8_5V: U4.14 (D)
- net PA9 is gone; now on net PA9_5V: U5.3 (A)
- net PB10 is gone; now on net PB10_5V: U1.6 (B)
- net PB5 is gone; now on net PB5_5V: U1.10 (C)
- net PB6 is gone; now on net PB6_5V: U1.14 (D)
- net PB8 is gone; now on net PB8_5V: U2.10 (C)
- net PB9 is gone; now on net PB9_5V: U2.14 (D)
- net PC0 is gone; now on net PC0_5V: U6.10 (C)
- net PC1 is gone; now on net PC1_5V: U6.14 (D)
- net PC10 is gone; now on net PC10_5V: U8.14 (D)
- net PC2 is gone; now on net PC2_5V: U7.3 (A)
- net PC3 is gone; now on net PC3_5V: U7.6 (B)
- net PC4 is gone; now on net PC4_5V: U7.10 (C)
- net PC5 is gone; now on net PC5_5V: U7.14 (D)
- net PC6 is gone; now on net PC6_5V: U8.3 (A)
- net PC7 is gone; now on net PC7_5V: U2.6 (B)
- net PC8 is gone; now on net PC8_5V: U8.6 (B)
- net PC9 is gone; now on net PC9_5V: U8.10 (C)
- net +15V: now also J3.1 (Pin_1)
- net +3V3: now also C1.1, J1.3 (Pin_3), J2.3 (Pin_3)
- net +5V: now also J1.1 (Pin_1), J2.1 (Pin_1); no longer C1.1
- net GND: now also J1.2 (Pin_2), J1.38 (Pin_38), J1.4 (Pin_4), J1.40 (Pin_40), J2.2 (Pin_2), J2.38 (Pin_38), J2.4 (Pin_4), J2.40 (Pin_40), J3.2 (Pin_2)
- net NC: now also J1.37 (Pin_37), J1.39 (Pin_39), J2.37 (Pin_37), J2.39 (Pin_39)
- net PA0_5V: now also J2.27 (Pin_27)
- net PA0_HIGH: now also J1.27 (Pin_27)
- net PA10_5V: now also J2.35 (Pin_35)
- net PA10_HIGH: now also J1.35 (Pin_35)
- net PA11_5V: now also J2.34 (Pin_34)
- net PA11_HIGH: now also J1.34 (Pin_34)
- net PA12_5V: now also J2.32 (Pin_32)
- net PA12_HIGH: now also J1.32 (Pin_32)
- net PA13_5V: now also J2.30 (Pin_30)
- net PA13_HIGH: now also J1.30 (Pin_30)
- net PA14_5V: now also J2.28 (Pin_28)
- net PA14_HIGH: now also J1.28 (Pin_28)
- net PA15_5V: now also J2.26 (Pin_26)
- net PA15_HIGH: now also J1.26 (Pin_26)
- net PA1_5V: now also J2.15 (Pin_15)
- net PA1_HIGH: now also J1.15 (Pin_15)
- net PA2_5V: now also J2.13 (Pin_13)
- net PA2_HIGH: now also J1.13 (Pin_13)
- net PA3_5V: now also J2.11 (Pin_11)
- net PA3_HIGH: now also J1.11 (Pin_11)
- net PA4_5V: now also J2.9 (Pin_9)
- net PA4_HIGH: now also J1.9 (Pin_9)
- net PA5_5V: now also J2.7 (Pin_7)
- net PA5_HIGH: now also J1.7 (Pin_7)
- net PA6_5V: now also J2.19 (Pin_19)
- net PA6_HIGH: now also J1.19 (Pin_19)
- net PA7_5V: now also J2.17 (Pin_17)
- net PA7_HIGH: now also J1.17 (Pin_17)
- net PA8_5V: now also J2.5 (Pin_5)
- net PA8_HIGH: now also J1.5 (Pin_5)
- net PA9_5V: now also J2.36 (Pin_36)
- net PA9_HIGH: now also J1.36 (Pin_36)
- net PB10_5V: now also J2.33 (Pin_33)
- net PB10_HIGH: now also J1.33 (Pin_33)
- net PB5_5V: now also J2.31 (Pin_31)
- net PB5_HIGH: now also J1.31 (Pin_31)
- net PB6_5V: now also J2.29 (Pin_29)
- net PB6_HIGH: now also J1.29 (Pin_29)
- net PB8_5V: now also J2.23 (Pin_23)
- net PB8_HIGH: now also J1.23 (Pin_23)
- net PB9_5V: now also J2.21 (Pin_21)
- net PB9_HIGH: now also J1.21 (Pin_21)
- net PC0_5V: now also J2.24 (Pin_24)
- net PC0_HIGH: now also J1.24 (Pin_24)
- net PC10_5V: now also J2.6 (Pin_6)
- net PC10_HIGH: now also J1.6 (Pin_6)
- net PC1_5V: now also J2.22 (Pin_22)
- net PC1_HIGH: now also J1.22 (Pin_22)
- net PC2_5V: now also J2.20 (Pin_20)
- net PC2_HIGH: now also J1.20 (Pin_20)
- net PC3_5V: now also J2.18 (Pin_18)
- net PC3_HIGH: now also J1.18 (Pin_18)
- net PC4_5V: now also J2.16 (Pin_16)
- net PC4_HIGH: now also J1.16 (Pin_16)
- net PC5_5V: now also J2.14 (Pin_14)
- net PC5_HIGH: now also J1.14 (Pin_14)
- net PC6_5V: now also J2.12 (Pin_12)
- net PC6_HIGH: now also J1.12 (Pin_12)
- net PC7_5V: now also J2.25 (Pin_25)
- net PC7_HIGH: now also J1.25 (Pin_25)
- net PC8_5V: now also J2.10 (Pin_10)
- net PC8_HIGH: now also J1.10 (Pin_10)
- net PC9_5V: now also J2.8 (Pin_8)
- net PC9_HIGH: now also J1.8 (Pin_8)
Other:
- note removed: "Morpho connector"
- moved on the sheet: C4

Commit message: Screw terminal adapter added
Parts:
- J3: footprint Connector_PinHeader_2.54mm:PinHeader_1x02_P2.54mm_Vertical -> TerminalBlock_Phoenix:TerminalBlock_Phoenix_PT-1,5-2-3.5-H_1x02_P3.50mm_Horizontal
Changed lines of the file:
@@
 F 0 "J3" H 12228 7576 50  0000 L CNN
 F 1 "Conn_01x02_Female" H 12228 7485 50  0000 L CNN
-F 2 "Connector_PinHeader_2.54mm:PinHeader_1x02_P2.54mm_Vertical" H 12200 7600 50  0001 C CNN
+F 2 "TerminalBlock_Phoenix:TerminalBlock_Phoenix_PT-1,5-2-3.5-H_1x02_P3.50mm_Horizontal" H 12200 7600 50  0001 C CNN
 F 3 "~" H 12200 7600 50  0001 C CNN
 	1    12200 7600
